File: 0016_Temperature_Humidity_Module_SHT31.kicad_sch (KiCad schematic)
At the start: 7 parts, among them U1 SHT31-DIS

Commit message: Add files via upload
Parts:
- removed R5: 0r, symbol Device:R
- added D1: LED, LED_SMD:LED_0805_2012Metric, symbol Device:LED
- added JP2: Jumper_3_Open, Jumper:SolderJumper-3_P1.3mm_Open_Pad1.0x1.5mm, symbol Jumper:Jumper_3_Open
- added U2: ~, Moduler_:pin_header, symbol moduler_pin:air
- C1: footprint (none) -> Capacitor_SMD:C_0805_2012Metric
- R1, R2, R3: footprint (none) -> Resistor_SMD:R_0805_2012Metric
- R4: value 10k -> 470r; footprint (none) -> Resistor_SMD:R_0805_2012Metric
Connections:
- net VCC is gone; now on net +3V3: C1.1, R1.1, R2.1, R3.1, U1.5 (VDD)
- net GND: now also D1.1 (K), JP2.3 (B), U2.9; no longer R4.2
- net INT: now also U2.13
- net RESET: now also U2.12
- net SCL: now also U2.5
- net SDA: now also U2.6
- net +3V3: now reaches R4.1
- net +3V3: now also JP2.1 (A), U2.8; no longer U1.2 (ADDR)
- new net: D1.2 (A), R4.2
- new net ADDR: JP2.2 (C), U1.2 (ADDR)
- no-connect marks 0 -> 12
Other:
- note added: "AIR PIN"
- note added: "I2C PULLUPS"
- note added: "SENSOR"
- moved on the sheet: C1, R2, R3, U1
